File: HW/ver. 1/HRM/HRM.kicad_pcb (KiCad board)
At the start: 2 copper layers, 38 x 90 mm, 113 parts, among them J1 USB_B_Micro, J10 Screw_Terminal_01x01, J11 Screw_Terminal_01x01, J12 Screw_Terminal_01x01, J2 BATT, J3 UART, J4 I2C, J5 EINK, J6 HSPI, J7 Door sensor, J8 ADC, J9 Screw_Terminal_01x01, Q1 PMOS-Si4403DDY, Q10 BSS84, Q11 BSS138, Q12 BC847, Q13 BC847, Q2 BSS138, Q3 BSS84, Q4 BSS84, Q5 BSS84, Q6 BSS138, Q7 BSS138, Q8 BSS138, Q9 BSS138, SW1 ON/OFF, U1 MCP73833, U2 TPS73733, U3 TPS3839K33, U4 ESP32-WROOM, U5 TPL5111, U6 LM4040-2.5, U7 FT231XS

Commit message: finished schema
Parts:
- removed D3: D, Mylib_Footprints:D0805
- removed J10, J11, J12: Screw_Terminal_01x01, Mylib_Footprints:Screwh_hole-2.5mm
- removed J5: EINK, Connector_PinHeader_2.54mm:PinHeader_1x08_P2.54mm_Vertical
- removed L1, L2: Ferite bead, Mylib_Footprints:R0805
- removed Q10: BSS84, Package_TO_SOT_SMD:SOT-23
- removed Q11, Q7, Q8, Q9: BSS138, Package_TO_SOT_SMD:SOT-23
- removed Q12, Q13: BC847, Package_TO_SOT_SMD:SOT-23
- added BTN4: user button, Mylib_Footprints:BTN_6x6mm, F.Cu at (63.2, 68.8)
- added BTN5: user button, Mylib_Footprints:BTN_6x6mm, F.Cu at (93.2, 37.9)
- added C30: 100n, Mylib_Footprints:C0805, F.Cu at (82.7, 69.5)
- added C31: 100n, Mylib_Footprints:C0805, F.Cu at (77.5, 75.0)
- added C32: 100n, Mylib_Footprints:C0805, F.Cu at (102.3, 50.3)
- added FB1: Ferite bead, Mylib_Footprints:R0805, F.Cu at (113.4, 36.7)
- added FB2: Ferite bead, Mylib_Footprints:R0805, F.Cu at (93.8, 57.7)
- added LED7: User, Mylib_Footprints:LED-THT-3.0mm, F.Cu at (101.4, 39.7)
- BTN1: value Push notification -> RESET; footprint Mylib_Footprints:SW_Tactile_SPST_Angled_PTS645Vx83-2LFS -> Mylib_Footprints:BTN_6x6mm
- BTN2: value RESET -> BOOT
- BTN3: value BOOT -> user button
- C10, C11, C12, C16, C21, C22, C23, C25, C27, C29, C3, C4, D2, Q3, R1, R15, R2, R29, R3, R30, R35, R5, R7, U6, U7: moved to F.Cu
- C15, C24: value 100n -> 1u; moved to F.Cu
- C17: value 1u -> 100n; moved to F.Cu
- C18, C19: value 100n -> 10p; moved to F.Cu
- C20: value 10u -> 1u; moved to F.Cu
- C26, C28: value 100n -> 10u; moved to F.Cu
- J3: value UART -> Electrodes; footprint Connector_PinHeader_2.54mm:PinHeader_1x04_P2.54mm_Vertical -> Connector_JST:JST_XH_S2B-XH-A_1x02_P2.50mm_Horizontal
- J4: value I2C -> HSPI; footprint Connector_PinHeader_2.54mm:PinHeader_1x04_P2.54mm_Vertical -> Connector_PinHeader_2.54mm:PinHeader_1x06_P2.54mm_Vertical
- J6: value HSPI -> Screw_Terminal_01x01; footprint Connector_PinHeader_2.54mm:PinHeader_1x06_P2.54mm_Vertical -> Mylib_Footprints:Screwh_hole-2.5mm
- J7: value Door sensor -> Screw_Terminal_01x01; footprint Connector_PinHeader_2.54mm:PinHeader_1x03_P2.54mm_Vertical -> Mylib_Footprints:Screwh_hole-2.5mm
- J8: value ADC -> Screw_Terminal_01x01; footprint Connector_PinHeader_2.54mm:PinHeader_1x05_P2.54mm_Vertical -> Mylib_Footprints:Screwh_hole-2.5mm
- LED3: value Awake -> TX
- LED4: value User -> RX
- LED5: value TX -> Awake
- LED6: value RX -> User
- Q4: value BSS84 -> BSS138; moved to F.Cu
- Q5: value BSS84 -> BC847
- Q6: value BSS138 -> BC847; moved to F.Cu
- R10: value 4k7 -> 100k
- R11: value 47k -> 10k
- R12: value 100k -> 13k
- R13: value 100k -> 5k; moved to F.Cu
- R14: value 10k -> 24k
- R16: value 270k -> 50k; moved to F.Cu
- R17: value 100 -> 0; moved to F.Cu
- R18: value 100k -> 10k; moved to F.Cu
- R19: value 10k -> 1k
- R20: value 124k -> 1k; moved to F.Cu
- R21, R27: value 10k -> 1k; moved to F.Cu
- R22: value 13k -> 4k7; moved to F.Cu
- R23: value 5k -> 50k; moved to F.Cu
- R24: value 1k -> 4k7
- R25: value 1k -> 10k
- R26: value 24k -> 1k; moved to F.Cu
- R28, R31: value 10k -> 4k7; moved to F.Cu
- R32, R33: value 1k -> 10k; moved to F.Cu
- R34: value 4k7 -> 10k; moved to F.Cu
- R4: value R -> 1.54k; moved to F.Cu
- R6: value R -> 69.8k; moved to F.Cu
- SW1: value ON/OFF -> Power
- U1: value MCP73833 -> MCP73833-MSOP; footprint Mylib_Footprints:DFN10-EP_3x3mm_P0.5mm_EP1.65x2.38mm -> Package_SO:MSOP-10_3x3mm_P0.5mm; moved to F.Cu
- U4: value ESP32-WROOM -> MAX8511; footprint Mylib_Footprints:ESP32-WROOM -> Mylib_Footprints:SC70-5pin
- U5: value TPL5111 -> ESP32-WROOM; footprint Package_TO_SOT_SMD:SOT-23-6 -> Mylib_Footprints:ESP32-WROOM; moved to F.Cu
- moved J1 102.0 mm to (147.3, 66.2), turned to 90 degrees
- moved R5 99.0 mm to (125.8, 31.2), turned to 0 degrees
- moved J2 98.5 mm to (147.1, 59.3), turned to 90 degrees
- moved R2 96.9 mm to (120.6, 34.3), turned to 0 degrees
- moved C10 91.1 mm to (115.4, 33.7), turned to 0 degrees
- moved SW1 89.8 mm to (143.0, 50.4), turned to 90 degrees
- moved C9 87.5 mm to (118.6, 43.9), turned to 0 degrees
- moved C11 84.4 mm to (108.2, 41.6), turned to 0 degrees
- moved C7 83.0 mm to (116.1, 28.1), turned to 0 degrees
- moved R11 81.6 mm to (118.6, 40.6), turned to 0 degrees
- moved C29 80.7 mm to (120.6, 31.3)
- moved R34 76.8 mm to (128.9, 40.6), turned to 0 degrees
- moved R1 76.7 mm to (107.5, 47.8), turned to 0 degrees
- moved C8 76.5 mm to (110.2, 33.7), turned to 0 degrees
- moved R30 73.0 mm to (123.7, 43.8), turned to 0 degrees
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Connections:
- BTN1 pad 1: /Timer_delay -> GNDD
- BTN1 pad 2: +BATT -> /RESET
- BTN2 pad 1: GND -> GNDD
- BTN2 pad 2: /RESET -> /BOOT
- BTN3 pad 2: /BOOT -> User_BTN1
- C1 pad 2: GND -> GNDD
- C10 pad 1: GND -> GNDD
- C11 pad 1: GND -> GNDD
- C12 pad 2: GND -> GNDD
- C13 pad 1: GND -> GNDD
- C14 pad 1: GND -> GNDD
- C14 pad 2: Net-(C14-Pad2) -> +3V3
- C15 pad 1: GND -> GNDD
- C15 pad 2: +BATT -> +1V8
- C16 pad 1: Net-(C16-Pad1) -> GNDD
- C16 pad 2: Net-(C16-Pad2) -> +5VA
- C17 pad 1: GND -> GNDD
- C17 pad 2: Net-(C17-Pad2) -> +5VA
- C18 pad 1: GND -> GNDA
- C18 pad 2: +3V3 -> Net-(C18-Pad2)
- C19 pad 1: GND -> Net-(C19-Pad1)
- C19 pad 2: +3V3 -> GNDA
- C2 pad 2: GND -> GNDD
- C20 pad 1: GND -> (no net)
- C20 pad 2: +5VA -> (no net)
- C21 pad 1: GND -> GNDD
- C21 pad 2: +5VA -> /RESET
- C22 pad 1: GND -> /VBUS_SENSE
- C22 pad 2: +3V3 -> GNDD
- C23 pad 1: GND -> GNDD
- C23 pad 2: +3V3 -> 3V3_IO
- C24 pad 1: GND -> GNDA
- C24 pad 2: +BATT -> (no net)
- C25 pad 1: GND -> GNDA
- C25 pad 2: /RESET -> +1V8
- C26 pad 1: /VBUS_SENSE -> GNDA
- C26 pad 2: GND -> +1V8
- C27 pad 1: GND -> GNDD
- C27 pad 2: 3V3_IO -> +3V3
- C28 pad 1: GND -> GNDD
- C28 pad 2: +BATT -> +3V3
- C29 pad 2: /BOOT -> User_BTN1
- C3 pad 2: GND -> GNDD
- C4 pad 2: GND -> GNDD
- C5 pad 1: GND -> GNDD
- C6 pad 1: GND -> GNDD
- C7 pad 1: GND -> GNDD
- C8 pad 1: GND -> GNDD
- C9 pad 1: GND -> GNDD
- D2 pad 2: GND -> GNDD
- J1 pad 5: GND -> GNDD
- J2 pad 1: GND -> GNDD
- J3 pad 1: GND -> Net-(J3-Pad1)
- J3 pad 2: /UART2_TX -> Net-(J3-Pad2)
- J4 pad 2: /I2C_SDA -> (no net)
- J4 pad 3: /I2C_SCL -> (no net)
- J4 pad 4: +3V3 -> (no net)
- J6 pad 1: GND -> (no net)
- J7 pad 1: GND -> (no net)
- J8 pad 1: GND -> (no net)
- LED3 pad 1: GND -> Net-(LED3-Pad1)
- LED3 pad 2: Net-(LED3-Pad2) -> 3V3_IO
- LED4 pad 1: GND -> Net-(LED4-Pad1)
- LED4 pad 2: Net-(LED4-Pad2) -> 3V3_IO
- LED5 pad 1: Net-(LED5-Pad1) -> GNDD
- LED5 pad 2: 3V3_IO -> Net-(LED5-Pad2)
- LED6 pad 1: Net-(LED6-Pad1) -> GNDD
- LED6 pad 2: 3V3_IO -> Net-(LED6-Pad2)
- Q2 pad 2: GND -> GNDD
- Q3 pad 1: Net-(C17-Pad2) -> Net-(Q3-Pad1)
- Q4 pad 1: Net-(Q4-Pad1) -> +3V3
- Q4 pad 2: +BATT -> GNDD
- Q4 pad 3: /Timer_delay -> Net-(Q3-Pad1)
- Q5 pad 2: +BATT -> /RTS
- Q5 pad 3: /EN_Reg_USB -> /RESET
- Q6 pad 1: Net-(C16-Pad1) -> Net-(Q6-Pad1)
- Q6 pad 2: GND -> /DTR
- Q6 pad 3: Net-(Q4-Pad1) -> /BOOT
- R10 pad 1: /EN_Reg_USB -> GNDD
- R10 pad 2: Net-(C14-Pad2) -> Net-(Q2-Pad1)
- R11 pad 1: Net-(C14-Pad2) -> +BATT
- R11 pad 2: /EN_Reg_Tim -> Net-(Q3-Pad1)
- R12 pad 1: GND -> BAT_ADC
- R12 pad 2: Net-(Q2-Pad1) -> Net-(Q3-Pad3)
- R13 pad 1: Net-(Q4-Pad1) -> V_ref
- R13 pad 2: +BATT -> +3V3
- R14 pad 1: Net-(Q5-Pad1) -> GNDD
- R14 pad 2: +BATT -> BAT_ADC
- R15 pad 1: /Ext_wake -> +3V3
- R15 pad 2: +3V3 -> GNDD
- R16 pad 1: Net-(C17-Pad2) -> Net-(C18-Pad2)
- R16 pad 2: /F_edge_det -> Net-(J3-Pad2)
- R17 pad 1: Net-(C16-Pad2) -> GNDA
- R17 pad 2: Net-(Q3-Pad3) -> GNDD
- R18 pad 1: GND -> /RESET
- R18 pad 2: Net-(C16-Pad1) -> +3V3
- R19 pad 1: GND -> Net-(LED5-Pad2)
- R19 pad 2: +5VA -> +3V3
- R20 pad 1: GND -> Net-(LED6-Pad2)
- R20 pad 2: /Timer_delay -> User_LED1
- R21 pad 1: +BATT -> Net-(LED7-Pad2)
- R21 pad 2: Net-(Q10-Pad1) -> User_LED2
- R22 pad 1: /BAT_ADC -> /VBUS_SENSE
- R22 pad 2: Net-(Q10-Pad3) -> +5VA
- R23 pad 1: /V_ref -> Net-(C19-Pad1)
- R23 pad 2: +3V3 -> Net-(J3-Pad1)
- R24 pad 1: Net-(LED3-Pad2) -> Net-(Q5-Pad1)
- R24 pad 2: +3V3 -> /DTR
- R25 pad 1: Net-(LED4-Pad2) -> GNDD
- R25 pad 2: /User_LED -> /VBUS_SENSE
- R26 pad 1: GND -> /TX_LED
- R26 pad 2: /BAT_ADC -> Net-(LED3-Pad1)
- R27 pad 1: /RESET -> /RX_LED
- R27 pad 2: +3V3 -> Net-(LED4-Pad1)
- R28 pad 2: GND -> I2C_SCL
- R29 pad 1: /VBUS_SENSE -> +3V3
- R29 pad 2: +5VA -> I2C_SDA
- R30 pad 1: Net-(Q12-Pad1) -> +3V3
- R30 pad 2: /DTR -> INTB
- R31 pad 1: GND -> Net-(Q6-Pad1)
- R31 pad 2: /VBUS_SENSE -> /RTS
- R32 pad 1: /TX_LED -> /BOOT
- R32 pad 2: Net-(LED5-Pad1) -> +3V3
- R33 pad 1: /RX_LED -> User_BTN1
- R33 pad 2: Net-(LED6-Pad1) -> +3V3
- R34 pad 1: Net-(Q13-Pad1) -> User_BTN2
- R34 pad 2: /RTS -> +3V3
- R35 pad 1: /BOOT -> User_BTN3
- R6 pad 1: GND -> GNDD
- R7 pad 1: GND -> GNDD
- TH1 pad 2: GND -> GNDD
- U1 pad 5: GND -> GNDD
- U2 pad 3: GND -> GNDD
- U2 pad 5: Net-(C14-Pad2) -> +BATT
- U2 pad 6: GND -> GNDD
- U3 pad 1: GND -> GNDD
- U4 pad 1: GND -> +3V3
- U4 pad 2: +3V3 -> GNDD
- U4 pad 3: /RESET -> +3V3
- U4 pad 4: /BAT_ADC -> (no net)
- U4 pad 5: /V_ref -> +1V8
- U5 pad 1: +BATT -> GNDD
- U5 pad 2: GND -> +3V3
- U5 pad 3: /Timer_delay -> /RESET
- U5 pad 4: /DONE -> BAT_ADC
- U5 pad 5: /EN_Reg_Tim -> V_ref
- U5 pad 6: +BATT -> (no net)
- U6 pad 1: /V_ref -> V_ref
- U6 pad 2: GND -> GNDD
- U7 pad 16: GND -> GNDD
- U7 pad 20: /UART0_RX -> (no net)
- U7 pad 4: /UART0_TX -> (no net)
- U7 pad 6: GND -> GNDD
Routing:
- net +3V3: track 224.3 -> 0.00 mm, vias 14 -> 0
- net +BATT: track 216.1 -> 0.00 mm, vias 2 -> 0
- net GND: track 131.7 -> 0.00 mm, vias 109 -> 0
- net +5VA: track 92.4 -> 0.00 mm, vias 12 -> 0
- net /BOOT: track 65.6 -> 0.00 mm, vias 5 -> 0
- net /EN_Reg_Tim: track 62.2 -> 0.00 mm, vias 3 -> 0
- net /HSPI_CLK: track 58.4 -> 0.00 mm, vias 1 -> 0
- net 3V3_IO: track 58.4 -> 0.00 mm
- net /ADC1_4: track 54.4 -> 0.00 mm, vias 4 -> 0
- net Net-(LED6-Pad1): track 53.8 -> 0.00 mm, vias 2 -> 0
- net /ADC1_6: track 50.4 -> 0.00 mm, vias 2 -> 0
- net /Timer_delay: track 49.7 -> 0.00 mm, vias 3 -> 0
- net Net-(LED1-Pad1): track 49.7 -> 0.00 mm, vias 1 -> 0
- net /UART0_RX: track 49.1 -> 0.00 mm, vias 3 -> 0
- net /USBDM: track 48.2 -> 0.00 mm
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- removed copper zone on B.Cu, net +5VA
- removed copper zone on F.Cu, net +5VA
- removed copper zone on B.Cu, net GND
- removed copper zone on F.Cu, net GND
- removed copper zone on F.Cu, net Net-(FB2-Pad1)
Other:
- board outline removed
- board text removed: "1"
- board text removed: "3V3"
- board text removed: "Awake"
- board text removed: "BUSY"
- board text removed: "CLK"
- board text removed: "CS0"
- board text removed: "Charged"
- board text removed: "Charging"
- board text removed: "DC"
- board text removed: "DIN"
- board text removed: "Designed by OBU"
- board text removed: "Door"
- board text removed: "ESP32 - IoT ver. 1.0"
- board text removed: "GND"
- board text removed: "GPIOs"
- board text removed: "HSPI"
- board text removed: "I2C"
- board text removed: "IO32"
- board text removed: "IO34"
- board text removed: "IO35"
- board text removed: "MISO"
- board text removed: "MOSI"
- board text removed: "Push"
- board text removed: "RST"
- board text removed: "RX"
- board text removed: "SCL"
- board text removed: "SDA"
- board text removed: "TX"
- board text removed: "UART"
- board text removed: "User"
- board text removed: "VBat"
- board text removed: "sig"
- board text removed: "~CS"

Commit message: one of last schematic updates
Parts:
- removed the C16 at (108.2, 38.5)
- removed the C17 at (97.1, 44.0)
- removed the C32 at (102.3, 50.3)
- removed the J7 at (103.2, 71.3)
- removed the R16 at (125.8, 34.3)
- removed the R18 at (113.4, 43.0)
- removed the R19 at (72.3, 73.7)
- removed the R29 at (114.5, 52.5)
- removed the R30 at (123.7, 43.8)
- added C18: 100n, Mylib_Footprints:C0805, B.Cu at (125.2, 122.8)
- added C20: 100n, Mylib_Footprints:C0805, B.Cu at (160.7, 115.3)
- added C29: 100n, Mylib_Footprints:C0805, B.Cu at (199.5, 124.1)
- added C30: 100n, Mylib_Footprints:C0805, B.Cu at (201.5, 124.1)
- added C34: 100n, Mylib_Footprints:C0805, B.Cu at (161.3, 128.7)
- added E1: ECG_N, Mylib_Footprints:Electrode, F.Cu at (200.8, 142.5)
- added E2: ECG_P, Mylib_Footprints:Electrode, F.Cu at (128.0, 142.5)
- added FB3: Ferite bead, Mylib_Footprints:R0805, F.Cu at (182.7, 148.5)
- added FB4: Ferite bead, Mylib_Footprints:R0805, B.Cu at (174.4, 147.9)
- added J10: Screw_Terminal_01x01, Mylib_Footprints:Screwh_hole-1.5mm, F.Cu at (158.1, 143.0)
- added J12: Screw_Terminal_01x01, Mylib_Footprints:Screwh_hole-1.5mm, F.Cu at (173.9, 143.0)
- added J13: Screw_Terminal_01x01, Mylib_Footprints:Screwh_hole-2.5mm, F.Cu at (212.5, 95.5)
- added J5: I2C, Connector_PinHeader_2.54mm:PinHeader_1x05_P2.54mm_Vertical, F.Cu at (134.4, 95.1)
- added J6: Screw_Terminal_01x01, Mylib_Footprints:Screwh_hole-1.5mm, F.Cu at (158.1, 152.0)
- added J8: Screw_Terminal_01x01, Mylib_Footprints:Screwh_hole-1.5mm, F.Cu at (173.9, 152.0)
- added R11: 50k, Mylib_Footprints:R0805, F.Cu at (157.4, 146.6)
- added R20: 4k7, Mylib_Footprints:R0805, B.Cu at (133.9, 99.7)
- added R21: 4k7, Mylib_Footprints:R0805, B.Cu at (135.9, 99.7)
- added R23: 4k7, Mylib_Footprints:R0805, F.Cu at (194.9, 123.1)
- added R28: 1k, Mylib_Footprints:R0805, B.Cu at (194.8, 98.8)
- added U8: FT231XS, Package_SO:SSOP-20_3.9x8.7mm_P0.635mm, B.Cu at (194.8, 122.2)
- C10, C11, C23, C31, C6, C7, Q3, Q4, Q5, Q6, R1, R2, R24, R3, R31, R32, R33, R34, R35, R5, R7, U1, U2, U6: moved to B.Cu
- C12, C2, C3, C4, C5, C8: footprint Mylib_Footprints:C0805 -> Mylib_Footprints:C1206; moved to B.Cu
- C15: value 1u -> DNP; footprint Mylib_Footprints:C0805 -> Mylib_Footprints:C0603
- C21: value 100n -> 1u
- C22, C25: value 100n -> 10u; footprint Mylib_Footprints:C0805 -> Mylib_Footprints:C1206
- C24: value 1u -> 100n
- C26, C28: value 10u -> 100n; moved to B.Cu
- C27: value 100n -> 10u; footprint Mylib_Footprints:C0805 -> Mylib_Footprints:C1206; moved to B.Cu
- C32: renamed from C29; moved to B.Cu
- C33: renamed from C30; moved to B.Cu
- J3: footprint Connector_JST:JST_XH_S2B-XH-A_1x02_P2.50mm_Horizontal -> Connector_PinHeader_2.54mm:PinHeader_1x02_P2.54mm_Vertical
- J4: value HSPI -> OLED; footprint Connector_PinHeader_2.54mm:PinHeader_1x06_P2.54mm_Vertical -> Mylib_Footprints:1.3_inch_OLED
- R13: renamed from R11; moved to B.Cu
- R14: renamed from R12; moved to B.Cu
- R15: renamed from R13; moved to B.Cu
- R17: renamed from R14; moved to B.Cu
- R18: renamed from R15; moved to B.Cu
- R19: renamed from R28; moved to B.Cu
- R22: value 4k7 -> 10k; moved to B.Cu
- U7: value FT231XS -> MAX86150; footprint Package_SO:SSOP-20_3.9x8.7mm_P0.635mm -> Mylib_Footprints:OLGA-22pin
- moved D1 148.6 mm to (198.0, 116.8)
- moved Q1 146.4 mm to (194.2, 103.2), turned to 180 degrees
- moved F1 145.9 mm to (201.2, 106.0), turned to 90 degrees
- moved Q6 135.9 mm to (171.3, 123.6), turned to 180 degrees
- moved U1 135.0 mm to (187.5, 101.9)
- moved J7 134.9 mm to (211.8, 150.8)
- moved J3 134.8 mm to (152.0, 149.2), turned to 180 degrees
- moved LED1 134.2 mm to (206.5, 96.0)
- moved U7 132.6 mm to (166.0, 148.8)
- moved C14 131.4 mm to (180.8, 148.5), turned to 270 degrees
- moved BTN4 130.0 mm to (177.3, 131.2)
- moved C24 128.6 mm to (170.1, 149.1), turned to 270 degrees
- moved LED3 128.2 mm to (189.1, 117.6), turned to 270 degrees
- moved C17 127.6 mm to (160.4, 149.6), turned to 270 degrees
- moved FB2 127.1 mm to (206.5, 116.4)
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- renumbered C18 to C16, C19 to C17, C20 to C19, J8 to J11, J6 to J7, R17 to R12, R23 to R16, R20 to R29, R21 to R30
Connections:
- BTN3 pad 1: GND -> GNDD
- BTN4 pad 1: GND -> GNDD
- BTN5 pad 1: GND -> GNDD
- C14 pad 2: +3V3 -> Net-(C14-Pad2)
- C15 pad 1: GNDD -> Net-(C15-Pad1)
- C15 pad 2: +1V8 -> Net-(C15-Pad2)
- C16 pad 2: Net-(C18-Pad2) -> Net-(C15-Pad2)
- C17 pad 1: Net-(C19-Pad1) -> Net-(C15-Pad1)
- C19 pad 1: (no net) -> Net-(C19-Pad1)
- C19 pad 2: (no net) -> Net-(C19-Pad2)
- C21 pad 1: GNDD -> GNDA
- C21 pad 2: /RESET -> Net-(C21-Pad2)
- C22 pad 1: /VBUS_SENSE -> GNDD
- C22 pad 2: GNDD -> +5VA
- C23 pad 2: 3V3_IO -> +5VA
- C24 pad 2: (no net) -> +1V8
- C26 pad 1: GNDA -> GNDD
- C26 pad 2: +1V8 -> Net-(C26-Pad2)
- C27 pad 2: +3V3 -> Net-(C26-Pad2)
- C28 pad 2: +3V3 -> /RESET
- C32 pad 1: GND -> GNDD
- C33 pad 1: GND -> GNDD
- J4 pad 1: GND -> GNDD
- J4 pad 2: (no net) -> +3V3
- J4 pad 3: (no net) -> OLED_CLK
- J4 pad 4: (no net) -> OLED_MOSI
- J4 pad 5: (no net) -> OLED_RES
- J4 pad 6: +3V3 -> OLED_DC
- R16 pad 1: Net-(C19-Pad1) -> Net-(C15-Pad1)
- R22 pad 1: /VBUS_SENSE -> /RESET
- R22 pad 2: +5VA -> +3V3
- U4 pad 1: +3V3 -> Net-(C14-Pad2)
- U4 pad 3: +3V3 -> Net-(C14-Pad2)
- U5 pad 27: (no net) -> OLED_RES
- U5 pad 28: (no net) -> OLED_DC
- U5 pad 29: (no net) -> OLED_CS
- U5 pad 30: (no net) -> OLED_CLK
- U5 pad 37: (no net) -> OLED_MOSI
- U7 pad 1: /DTR -> (no net)
- U7 pad 10: /RX_LED -> (no net)
- U7 pad 11: /USBDP -> (no net)
- U7 pad 12: /USBDM -> (no net)
- U7 pad 13: 3V3_IO -> +1V8
- U7 pad 14: 3V3_IO -> +1V8
- U7 pad 15: +5VA -> Net-(C26-Pad2)
- U7 pad 17: /TX_LED -> GNDA
- U7 pad 18: /VBUS_SENSE -> GNDA
- U7 pad 19: (no net) -> Net-(C21-Pad2)
- U7 pad 2: /RTS -> (no net)
- U7 pad 20: (no net) -> Net-(C19-Pad1)
- U7 pad 3: 3V3_IO -> (no net)
- U7 pad 4: (no net) -> Net-(C15-Pad2)
- U7 pad 5: (no net) -> Net-(C15-Pad1)
- U7 pad 6: GNDD -> (no net)
- U7 pad 7: (no net) -> INTB
- U7 pad 8: (no net) -> I2C_SDA
- U7 pad 9: (no net) -> I2C_SCL
Other:
- board outline added: 100 x 60 mm
- board text added: "1"

Commit message: Design of PCB
Parts:
- removed the BTN2 at (135.0, 124.6)
- removed C15: DNP, Mylib_Footprints:C0603
- removed the LED6 at (189.1, 124.1)
- removed Q3: BSS84, Package_TO_SOT_SMD:SOT-23
- removed Q4: BSS138, Package_TO_SOT_SMD:SOT-23
- removed R13, R18: 10k, Mylib_Footprints:R0805
- added BTN4: BOOT, Mylib_Footprints:BTN_6x6mm, F.Cu at (135.0, 124.6)
- added LED1: User, Mylib_Footprints:LED-THT-3.0mm, F.Cu at (189.1, 128.9)
- E1: value ECG_N -> ECG_P
- E2: value ECG_P -> ECG_N
- R26, R27, R29, R30: moved to B.Cu
- moved FB3 35.2 mm to (147.8, 143.8), turned to 270 degrees
- moved C14 31.4 mm to (149.7, 143.8), turned to 90 degrees
- moved R29 30.6 mm to (159.7, 120.6)
- moved R30 30.6 mm to (159.7, 118.5)
- moved J3 28.9 mm to (180.8, 150.9), turned to 270 degrees
- moved U4 25.0 mm to (152.9, 144.0), turned to 0 degrees
- moved R12 22.6 mm to (154.9, 146.5), turned to 180 degrees
- moved J8 20.5 mm to (157.0, 140.3), turned to 180 degrees
- moved FB4 18.7 mm to (156.1, 144.4), turned to 90 degrees
- moved J6 18.1 mm to (172.0, 140.3), turned to 180 degrees
- moved J12 17.9 mm to (157.0, 148.8), turned to 180 degrees
- moved R16 15.2 mm to (171.6, 143.5), turned to 0 degrees
- moved J10 15.0 mm to (172.0, 148.8), turned to 180 degrees
- moved C25 14.5 mm to (158.3, 144.4), turned to 90 degrees
- moved C27 14.4 mm to (158.2, 144.5), turned to 90 degrees
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- renumbered BTN3 to BTN1, BTN5 to BTN2, BTN4 to BTN3, BTN1 to BTN5, LED7 to LED2, LED1 to LED6, LED2 to LED7
Connections:
- BTN2 pad 2: User_BTN3 -> User_BTN2
- BTN3 pad 2: User_BTN2 -> User_BTN3
- C33 pad 2: User_BTN2 -> User_BTN3
- C34 pad 2: User_BTN3 -> User_BTN2
- J3 pad 1: Net-(E2-Pad1) -> Net-(E1-Pad1)
- J3 pad 2: Net-(E1-Pad1) -> Net-(E2-Pad1)
- R11 pad 2: Net-(E1-Pad1) -> Net-(E2-Pad1)
- R14 pad 2: Net-(Q3-Pad3) -> +BATT
- R16 pad 2: Net-(E2-Pad1) -> Net-(E1-Pad1)
- R34 pad 1: User_BTN2 -> User_BTN3
- R35 pad 1: User_BTN3 -> User_BTN2
Routing:
- net +3V3: track 0.00 -> 234.8 mm, vias 0 -> 9
- net I2C_SDA: track 0.00 -> 91.6 mm, vias 0 -> 2
- net INTB: track 0.00 -> 89.8 mm, vias 0 -> 3
- net I2C_SCL: track 0.00 -> 88.6 mm, vias 0 -> 2
- net /BOOT: track 0.00 -> 87.7 mm, vias 0 -> 6
- net /RESET: track 0.00 -> 80.9 mm, vias 0 -> 3
- net +5VA: track 0.00 -> 67.4 mm, vias 0 -> 2
- net Net-(E2-Pad1): track 0.00 -> 63.1 mm
- net User_BTN3: track 0.00 -> 61.5 mm, vias 0 -> 2
- net User_BTN2: track 0.00 -> 56.7 mm, vias 0 -> 2
- net User_BTN1: track 0.00 -> 54.7 mm, vias 0 -> 2
- net OLED_MOSI: track 0.00 -> 47.8 mm
- net OLED_CS: track 0.00 -> 42.1 mm, vias 0 -> 1
- net BAT_ADC: track 0.00 -> 40.5 mm, vias 0 -> 1
- net Net-(E1-Pad1): track 0.00 -> 39.8 mm
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- added copper zone on B.Cu, net +5VA
- added copper zone on B.Cu, net +BATT
- added copper zone on F.Cu, net +BATT
- added copper zone on B.Cu, net GNDA
- added copper zone on F.Cu, net GNDA
- added copper zone on B.Cu, net GNDD
- added copper zone on F.Cu, net GNDD
- added copper zone on B.Cu, net Net-(C12-Pad1)
- added copper zone on F.Cu, net Net-(C12-Pad1)
- added copper zone on F.Cu, net Net-(C13-Pad2)
- added copper zone on F.Cu, net Net-(C14-Pad2)
Other:
- board text added: "BOOT"
- board text added: "Charged"
- board text added: "Charging"
- board text added: "Designed by OBU"
- board text added: "HRM device - ver. 1.0"
- board text added: "MAX86150 sensor"
- board text added: "ON"
- board text added: "RESET"
- board text added: "Rx"
- board text added: "Tx"
