File: HW/ver. 1/HRM/HRM.sch (KiCad schematic (older format))
At the start: 108 parts, among them J1 USB_B_Micro, J10 Screw_Terminal_01x01, J11 Screw_Terminal_01x01, J12 Screw_Terminal_01x01, J2 BATT, J6 HSPI, J9 Screw_Terminal_01x01, Q1 PMOS-Si4403DDY, Q10 BSS84, Q11 BSS138, Q12 BC847, Q13 BC847, Q2 BSS138, U1 MCP73833, U2 TPS73733, U3 TPS3839K33, U4 ESP32-WROOM, U6 LM4040-2.5, U7 FT231XS

Commit message: Added labels on MCU pins
Parts:
- removed U1: MCP73833, Mylib_Footprints:DFN10-EP_3x3mm_P0.5mm_EP1.65x2.38mm, symbol MyLib-Power_Management:MCP73833
- added U?: MCP73833-MSOP, symbol MyLib-Power_Management:MCP73833-MSOP
Connections:
- net labels added: OLED_CLK, OLED_CS, OLED_DC, OLED_MOSI, OLED_RES, UART_RX, UART_TX, User_btn
- net labels removed: ADC1_4, ADC1_6, ADC1_7, DONE, EINK_BUSY, EINK_CLK, EINK_CS, EINK_DC, EINK_DIN, EN_Reg_Tim, Ext_wake, UART2_RX, UART2_TX, VSPI_MISO, user_btn
- wire segments 354 -> 336
Other:
- moved on the sheet: BTN2, BTN3, BTN?, C20, C21, C23, C25, C26, C27, C29, C?, J6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

Commit message: finished schema
Parts:
- removed C23, C?: 100n, Mylib_Footprints:C0805, symbol Device:C
- removed C?: 10u, Mylib_Footprints:C0805, symbol Device:C
- removed FB?: Ferite bead, Mylib_Footprints:R0805, symbol Device:L_Core_Ferrite
- removed R?: 0, symbol Device:R
- added BTN4, BTN5: user button, Mylib_Footprints:BTN_6x6mm, symbol Switch:SW_Push
- added C30, C32: 100n, Mylib_Footprints:C0805, symbol Device:C
- added LED7: User, Mylib_Footprints:LED-THT-3.0mm, symbol Device:LED
- added R21: 1k, Mylib_Footprints:R0805, symbol Device:R
- added R34, R35: 10k, Mylib_Footprints:R0805, symbol Device:R
- J4: renamed from J6; value HSPI -> OLED; symbol Connector:Screw_Terminal_01x06 -> Connector:Screw_Terminal_01x07
- R16, R17, R23, R28, R29, R30: renamed from R?; footprint (none) -> Mylib_Footprints:R0805
- R4: value R -> 1.54k
- R6: value R -> 69.8k
- SW1: renamed from SW?; footprint (none) -> Mylib_Footprints:Switch_P-KNX125
- U1: renamed from U?; footprint (none) -> Package_SO:MSOP-10_3x3mm_P0.5mm
- U4: renamed from U?; footprint (none) -> Mylib_Footprints:SC70-5pin
- gave numbers to parts that had none: 17
- renumbered BTN2 to BTN1, BTN3 to BTN2, C20 to C16, C21 to C17, C25 to C21, C26 to C22, C27 to C23, C29 to C31, J9 to J6, J10 to J7, J11 to J8, J12 to J9, LED5 to LED3, LED6 to LED4, LED3 to LED5, LED4 to LED6, Q10 to Q3, Q11 to Q4, Q12 to Q5, Q13 to Q6, R12 to R10, R21 to R11, R22 to R12, R23 to R13, R26 to R14, R28 to R15, R27 to R18, R24 to R19, R25 to R20, R29 to R22, R30 to R24, R31 to R25, R32 to R26, R33 to R27, R34 to R31, R35 to R32, R14 to R33, U4 to U5
Connections:
- net HSPI_CLK is gone; now on net +3V3: J4.2 (Pin_2)
- net HSPI_CS0 is gone; now on net OLED_CLK: J4.3 (Pin_3)
- net HSPI_MISO is gone; now on net OLED_MOSI: J4.4 (Pin_4)
- net HSPI_MOSI is gone; now on net OLED_RES: J4.5 (Pin_5)
- net User_btn is gone; now on net User_BTN1: BTN3.2, C29.2, R33.1
- net +1V8: now also C25.2, C26.2, U8.13 (VDD_DIG)
- net +3V3: now also R34.2, R35.2; no longer J4.6 (Pin_6), R20.2
- net GND: now also BTN4.1, BTN5.1, C30.1, C32.1; no longer J4.1 (Pin_1)
- net GNDA: now also C25.1, C26.1, U8.17 (GND_D)
- net GNDD: now also J4.1 (Pin_1), LED6.1 (K), LED7.1 (K)
- net GNDREF: no longer C25.1, C26.1, U8.17 (GND_D)
- net INTB: now also U5.26 (IO4)
- net OLED_CLK: now also U5.30 (VSPI_CLK/IO18)
- net OLED_CS: now also J4.7 (Pin_7), U5.29 (VSPI_CS/IO5)
- net OLED_DC: now also J4.6 (Pin_6), U5.28 (IO17)
- net OLED_MOSI: now also U5.37 (VSPI_MOSI/IO23)
- net OLED_RES: now also U5.27 (IO16)
- net User_LED1: now reaches U5.10 (IO25)
- net User_LED1: now also R20.2
- net User_LED2: now reaches U5.11 (IO26)
- net User_LED2: now also R21.2
- net User_BTN1: now reaches U5.7 (IO35)
- net User_BTN2: now reaches U5.8 (IO32)
- net User_BTN2: now also BTN4.2, C30.2, R34.1
- net User_BTN3: now reaches U5.9 (IO33)
- net User_BTN3: now also BTN5.2, C32.2, R35.1
- net User_LED: no longer names the net of U5.24 (IO2)
- net User_LED: no longer LED6.1 (K)
- new net: LED7.2 (A), R21.1
Other:
- moved on the sheet: BTN1, BTN2, BTN3, C16, C17, C18, C19, C20, C21, C22, C23, C24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

Commit message: one of last schematic updates
Parts:
- removed C32: 100n, Mylib_Footprints:C0805, symbol Device:C
- added C18, C20, C34: 100n, Mylib_Footprints:C0805, symbol Device:C
- added FB3, FB4: Ferite bead, Mylib_Footprints:R0805, symbol Device:Ferrite_Bead_Small
- added J10, J12, J6, J8: Screw_Terminal_01x01, Mylib_Footprints:Screwh_hole-1.5mm, symbol Connector:Screw_Terminal_01x01
- C12, C2, C3, C4, C5, C8: footprint Mylib_Footprints:C0805 -> Mylib_Footprints:C1206
- C15: value 1u -> DNP; footprint Mylib_Footprints:C0805 -> Mylib_Footprints:C0603
- C22: renamed from C16; footprint Mylib_Footprints:C0805 -> Mylib_Footprints:C1206
- C25: renamed from C26; footprint Mylib_Footprints:C0805 -> Mylib_Footprints:C1206
- C27: renamed from C28; footprint Mylib_Footprints:C0805 -> Mylib_Footprints:C1206
- E1: renamed from TP1; footprint (none) -> Mylib_Footprints:Electrode
- E2: renamed from TP2; footprint (none) -> Mylib_Footprints:Electrode
- FB1, FB2: symbol Device:L_Core_Ferrite -> Device:Ferrite_Bead_Small
- J3: footprint Connector_JST:JST_XH_S2B-XH-A_1x02_P2.50mm_Horizontal -> Connector_PinHeader_2.54mm:PinHeader_1x02_P2.54mm_Vertical
- J4: footprint Connector_PinHeader_2.54mm:PinHeader_1x06_P2.54mm_Vertical -> Mylib_Footprints:1.3_inch_OLED
- J5: footprint (none) -> Connector_PinHeader_2.54mm:PinHeader_1x05_P2.54mm_Vertical
- U7: renamed from U8; footprint (none) -> Mylib_Footprints:OLGA-22pin
- renumbered C18 to C16, C19 to C17, C20 to C19, C24 to C21, C17 to C23, C25 to C24, C27 to C26, C21 to C28, C22 to C29, C23 to C30, C29 to C32, C30 to C33, J8 to J11, J9 to J13, J6 to J7, J7 to J9, R16 to R11, R17 to R12, R11 to R13, R12 to R14, R13 to R15, R23 to R16, R14 to R17, R15 to R18, R28 to R19, R29 to R20, R30 to R21, R18 to R22, R22 to R23, R19 to R28, R20 to R29, R21 to R30, U7 to U8
Connections:
- net GND is gone; now on net GNDD: BTN3.1, BTN4.1, BTN5.1, C32.1, C33.1
- net GNDREF is gone; now on net GNDD: J5.1 (Pin_1)
- net +1V8: no longer C15.2
- net +3V3: now also C18.2, FB3.2, FB4.1; no longer C14.2, C26.2, C27.2, U4.1 (IN), U4.3 (~SHDN), U7.15 (VLED)
- net BAT_ADC: now also C20.2
- net GNDD: now also C18.1, C20.1, C34.1; no longer C15.1
- net User_BTN3: now also C34.2
- net at C16.2, R11.1, U7.4 (ECG_N): now also C15.2
- net at C17.1, R16.1, U7.5 (ECG_P): now also C15.1
- new net: C26.2, C27.2, FB4.2, U7.15 (VLED)
- new net: C14.2, FB3.1, U4.1 (IN), U4.3 (~SHDN)
- no-connect marks 18 -> 22
Other:
- moved on the sheet: C16, C17, E1, E2, J3, R11, R15, R16, U6

Commit message: Design of PCB
Parts:
- removed C15: DNP, Mylib_Footprints:C0603, symbol Device:C
- removed Q3: BSS84, Package_TO_SOT_SMD:SOT-23, symbol Transistor_FET:BSS84
- removed Q4: BSS138, Package_TO_SOT_SMD:SOT-23, symbol Transistor_FET:BSS138
- removed R13, R18: 10k, Mylib_Footprints:R0805, symbol Device:R
- E1: value ECG_N -> ECG_P
- E2: value ECG_P -> ECG_N
- R7: value 1k -> 2k
- renumbered BTN3 to BTN1, BTN5 to BTN2, BTN4 to BTN3, BTN2 to BTN4, BTN1 to BTN5, LED6 to LED1, LED7 to LED2, LED1 to LED6, LED2 to LED7
Connections:
- net +BATT: now also R14.2
- net User_BTN2: now also BTN2.2, C34.2, R35.1; no longer BTN3.2, C33.2, R34.1
- net User_BTN3: now also BTN3.2, C33.2, R34.1; no longer BTN2.2, C34.2, R35.1
- net at J3.2 (Pin_2), R11.2: now also E2.1; no longer E1.1
- net at J3.1 (Pin_1), R16.2: now also E1.1; no longer E2.1
Other:
- note added: "500 mA"
- note added: "no need for output capacitor\n(regulator is close to the sensor)"
- moved on the sheet: BTN1, BTN2, BTN3, C12, C14, C16, C17, C18, C20, C32, C33, C34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
